File: openautov1point2.sch (EAGLE design)
At the start: 80 parts, among them CN1 6p-2.54, CN2 6p-2.54, CN3 6p-2.54, CN4 3p-2.54, CN5 3p-2.54, IC1 NC7SZ14M5X, IC2 TJA1049, IC3 NCP1117CORRECT, J3 4p-2.54, Q1 s9013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

Commit message: added fiducials to PCB, created case
Parts:
- added FID1, FID2, FID3, FID4: FIDUCIAL1.5X3, SparkFun-Retired:FIDUCIAL1.5X3
Changed lines of the file:
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@@
 <part name="CN5" library="Seeed-Connector" deviceset="DIP-BLACK-MALE-HEADER-VERT(3P-2.54)" device="" value="3p-2.54"/>
 <part name="U$10" library="Power or GND " deviceset="GND_POWER" device=""/>
+<part name="FID1" library="SparkFun-Retired" deviceset="FIDUCIAL" device="1.5X3"/>
+<part name="FID2" library="SparkFun-Retired" deviceset="FIDUCIAL" device="1.5X3"/>
+<part name="FID3" library="SparkFun-Retired" deviceset="FIDUCIAL" device="1.5X3"/>
+<part name="FID4" library="SparkFun-Retired" deviceset="FIDUCIAL" device="1.5X3"/>
 </parts>
 <sheets>
@@
 <instance part="CN5" gate="G$1" x="386.08" y="-39.37" rot="R90"/>
 <instance part="U$10" gate="G$1" x="382.27" y="-48.26"/>
+<instance part="FID1" gate="G$1" x="109.22" y="-111.76"/>
+<instance part="FID2" gate="G$1" x="114.3" y="-111.76"/>
+<instance part="FID3" gate="G$1" x="119.38" y="-111.76"/>
+<instance part="FID4" gate="G$1" x="124.46" y="-111.76"/>
 </instances>
 <busses>
