File: openautov1point2.brd (EAGLE design)
At the start: 97 x 77 mm, 80 parts, among them CN1 6p-2.54, CN2 6p-2.54, CN3 6p-2.54, CN4 3p-2.54, CN5 3p-2.54, IC1 NC7SZ14M5X, IC2 TJA1049, IC3 NCP1117CORRECT, J3 4p-2.54, Q1 s9013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

Commit message: added fiducials to PCB, created case
Parts:
- added FID1, FID2, FID3, FID4: FIDUCIAL1.5X3, SparkFun-Retired:FIDUCIAL-1.5X3
Changed lines of the file:
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@@
 <element name="C14" library="Seeed-Capacitor" package="C0603" value="100nf" x="76" y="10" smashed="yes" rot="R270">
 <attribute name="MPN" value="CC0603KRX7R9BB104" x="76" y="10" size="1.778" layer="27" rot="R270" display="off"/>
+<attribute name="NAME" x="75" y="12" size="0.889" layer="25" ratio="11"/>
 <attribute name="NAME" x="77.27" y="10.254" size="0.635" layer="33" ratio="10" rot="R180"/>
-<attribute name="NAME" x="75" y="12" size="0.889" layer="25" ratio="11"/>
 <attribute name="VALUE" x="76" y="11" size="0.635" layer="27" ratio="10"/>
 </element>
 <element name="C16" library="Seeed-Capacitor" package="C0603" value="100nf" x="40" y="70" smashed="yes" rot="R180">
 <attribute name="MPN" value="CC0603KRX7R9BB104" x="40" y="70" size="1.778" layer="27" rot="R180" display="off"/>
+<attribute name="NAME" x="39" y="72" size="0.889" layer="25" ratio="11" rot="R90"/>
 <attribute name="NAME" x="40.254" y="68.73" size="0.635" layer="33" ratio="10" rot="R90"/>
-<attribute name="NAME" x="39" y="72" size="0.889" layer="25" ratio="11" rot="R90"/>
 <attribute name="VALUE" x="40" y="72" size="0.635" layer="27" ratio="10" rot="R90"/>
 </element>
 <element name="C17" library="Seeed-Capacitor" package="C0603" value="10pf" x="44" y="63" smashed="yes" rot="R90">
 <attribute name="MPN" value="CC0603JRNPO9BN100" x="44" y="63" size="1.778" layer="27" rot="R90" display="off"/>
+<attribute name="NAME" x="40" y="64" size="0.889" layer="25" ratio="11"/>
 <attribute name="NAME" x="42.73" y="62.746" size="0.635" layer="33" ratio="10"/>
-<attribute name="NAME" x="40" y="64" size="0.889" layer="25" ratio="11"/>
 <attribute name="VALUE" x="40" y="63" size="0.635" layer="27" ratio="10"/>
 </element>
 <element name="C18" library="Seeed-Capacitor" package="C0603" value="10pf" x="48" y="63" smashed="yes" rot="R270">
 <attribute name="MPN" value="CC0603JRNPO9BN100" x="48" y="63" size="1.778" layer="27" rot="R270" display="off"/>
+<attribute name="NAME" x="52" y="64" size="0.889" layer="25" ratio="11" rot="R180"/>
 <attribute name="NAME" x="49.27" y="63.254" size="0.635" layer="33" ratio="10" rot="R180"/>
-<attribute name="NAME" x="52" y="64" size="0.889" layer="25" ratio="11" rot="R180"/>
 <attribute name="VALUE" x="52" y="63" size="0.635" layer="27" ratio="10" rot="R180"/>
 </element>
 <element name="C19" library="Seeed-Capacitor" package="C0603" value="100nf" x="39" y="56" smashed="yes" rot="R180">
 <attribute name="MPN" value="CC0603KRX7R9BB104" x="39" y="56" size="1.778" layer="27" rot="R180" display="off"/>
+<attribute name="NAME" x="39.411" y="52.03" size="0.889" layer="25" ratio="11" rot="R90"/>
 <attribute name="NAME" x="39.254" y="54.73" size="0.635" layer="33" ratio="10" rot="R90"/>
-<attribute name="NAME" x="39.411" y="52.03" size="0.889" layer="25" ratio="11" rot="R90"/>
 <attribute name="VALUE" x="40.5875" y="54.73" size="0.635" layer="27" ratio="10" rot="R90"/>
 </element>
 <element name="C21" library="Seeed-Capacitor" package="C0603" value="10UF 6.3V" x="36" y="60" smashed="yes" rot="R180">
 <attribute name="MPN" value="CC0603MRX5R5BB106" x="36" y="60" size="1.778" layer="27" rot="R180" display="off"/>
+<attribute name="NAME" x="35.111" y="58.73" size="0.889" layer="25" ratio="11" rot="R90"/>
 <attribute name="NAME" x="36.254" y="58.73" size="0.635" layer="33" ratio="10" rot="R90"/>
-<attribute name="NAME" x="35.111" y="58.73" size="0.889" layer="25" ratio="11" rot="R90"/>
 <attribute name="VALUE" x="37.5875" y="58.73" size="0.635" layer="27" ratio="10" rot="R90"/>
 </element>
 <element name="C22" library="Seeed-Capacitor" package="C0603" value="100nf" x="46" y="70" smashed="yes" rot="R180">
 <attribute name="MPN" value="CC0603KRX7R9BB104" x="46" y="70" size="1.778" layer="27" rot="R180" display="off"/>
+<attribute name="NAME" x="46" y="72" size="0.889" layer="25" ratio="11" rot="R90"/>
 <attribute name="NAME" x="46.254" y="68.73" size="0.635" layer="33" ratio="10" rot="R90"/>
-<attribute name="NAME" x="46" y="72" size="0.889" layer="25" ratio="11" rot="R90"/>
 <attribute name="VALUE" x="47" y="72" size="0.635" layer="27" ratio="10" rot="R90"/>
 </element>
@@
 <element name="C6" library="Seeed-Capacitor" package="C0603" value="10UF 6.3V" x="72" y="69" smashed="yes">
 <attribute name="MPN" value="CC0603MRX5R5BB106" x="72" y="69" size="1.778" layer="27" display="off"/>
+<attribute name="NAME" x="69" y="69" size="0.889" layer="25" ratio="11" rot="R270"/>
 <attribute name="NAME" x="71.746" y="70.27" size="0.635" layer="33" ratio="10" rot="R270"/>
-<attribute name="NAME" x="69" y="69" size="0.889" layer="25" ratio="11" rot="R270"/>
 <attribute name="VALUE" x="70" y="70" size="0.635" layer="27" ratio="10" rot="R270"/>
 </element>
@@
 <element name="C8" library="Seeed-Capacitor" package="C0603" value="100nf" x="72" y="73" smashed="yes">
 <attribute name="MPN" value="CC0603KRX7R9BB104" x="72" y="73" size="1.778" layer="27" display="off"/>
+<attribute name="NAME" x="69" y="73" size="0.889" layer="25" ratio="11" rot="R270"/>
 <attribute name="NAME" x="71.746" y="74.27" size="0.635" layer="33" ratio="10" rot="R270"/>
-<attribute name="NAME" x="69" y="73" size="0.889" layer="25" ratio="11" rot="R270"/>
 <attribute name="VALUE" x="70" y="74" size="0.635" layer="27" ratio="10" rot="R270"/>
 </element>
 <element name="C9" library="Seeed-Capacitor" package="C0603" value="100nf" x="93" y="60" smashed="yes" rot="R180">
 <attribute name="MPN" value="CC0603KRX7R9BB104" x="93" y="60" size="1.778" layer="27" rot="R180" display="off"/>
+<attribute name="NAME" x="95" y="59" size="0.889" layer="25" ratio="11" rot="R90"/>
 <attribute name="NAME" x="93.254" y="58.73" size="0.635" layer="33" ratio="10" rot="R90"/>
-<attribute name="NAME" x="95" y="59" size="0.889" layer="25" ratio="11" rot="R90"/>
 <attribute name="VALUE" x="96" y="59" size="0.635" layer="27" ratio="10" rot="R90"/>
 </element>
@@
 <element name="CN1" library="Seeed-Connector" package="H6-2.54" value="6p-2.54" x="10.45" y="65.63" smashed="yes" rot="R90">
 <attribute name="MPN" value="F185-1106A1BSYC1" x="10.45" y="65.63" size="1.778" layer="27" rot="R90" display="off"/>
+<attribute name="NAME" x="3.355" y="63.725" size="0.889" layer="25" ratio="11" rot="R180"/>
 <attribute name="NAME" x="12.99" y="66.265" size="0.635" layer="33" ratio="10" rot="R180"/>
-<attribute name="NAME" x="3.355" y="63.725" size="0.889" layer="25" ratio="11" rot="R180"/>
 <attribute name="VALUE" x="5.355" y="62.17" size="0.889" layer="27" ratio="11" rot="R180"/>
 </element>
 <element name="CN2" library="Seeed-Connector" package="H6-2.54" value="6p-2.54" x="29.55" y="70.72" smashed="yes" rot="R270">
 <attribute name="MPN" value="F185-1106A1BSYC1" x="29.55" y="70.72" size="1.778" layer="27" rot="R270" display="off"/>
+<attribute name="NAME" x="28" y="74" size="0.889" layer="25" ratio="11"/>
 <attribute name="NAME" x="27.01" y="70.085" size="0.635" layer="33" ratio="10"/>
-<attribute name="NAME" x="28" y="74" size="0.889" layer="25" ratio="11"/>
 <attribute name="VALUE" x="28" y="73" size="0.889" layer="27" ratio="11"/>
 </element>
 <element name="CN3" library="Seeed-Connector" package="H6-2.54" value="6p-2.54" x="29.55" y="55.07" smashed="yes" rot="R270">
 <attribute name="MPN" value="F185-1106A1BSYC1" x="29.55" y="55.07" size="1.778" layer="27" rot="R270" display="off"/>
+<attribute name="NAME" x="23.345" y="56.675" size="0.889" layer="25" ratio="11"/>
 <attribute name="NAME" x="27.01" y="54.435" size="0.635" layer="33" ratio="10"/>
-<attribute name="NAME" x="23.345" y="56.675" size="0.889" layer="25" ratio="11"/>
 <attribute name="VALUE" x="27.645" y="52.53" size="0.889" layer="27" ratio="11"/>
 </element>
@@
 <element name="D5" library="Seeed-Diode" package="SOD-123" value="20V-1A" x="53" y="71" smashed="yes" rot="R90">
 <attribute name="MPN" value="B5819W" x="53" y="71" size="1.778" layer="27" rot="R90" display="off"/>
+<attribute name="NAME" x="51.857" y="69.095" size="0.889" layer="25" ratio="11" rot="R90"/>
 <attribute name="NAME" x="53.635" y="70.111" size="0.381" layer="33" ratio="10" rot="R90"/>
-<attribute name="NAME" x="51.857" y="69.095" size="0.889" layer="25" ratio="11" rot="R90"/>
 <attribute name="VALUE" x="55.032" y="69.095" size="0.889" layer="27" font="vector" ratio="11" rot="R90"/>
 </element>
 <element name="D6" library="Seeed-Diode" package="SOD-123" value="20V-1A" x="50" y="71" smashed="yes" rot="R90">
 <attribute name="MPN" value="B5819W" x="50" y="71" size="1.778" layer="27" rot="R90" display="off"/>
+<attribute name="NAME" x="48.857" y="69.095" size="0.889" layer="25" ratio="11" rot="R90"/>
 <attribute name="NAME" x="50.635" y="70.111" size="0.381" layer="33" ratio="10" rot="R90"/>
-<attribute name="NAME" x="48.857" y="69.095" size="0.889" layer="25" ratio="11" rot="R90"/>
 <attribute name="VALUE" x="52.032" y="69.095" size="0.889" layer="27" font="vector" ratio="11" rot="R90"/>
 </element>
@@
 <attribute name="VALUE" x="82" y="57" size="0.889" layer="27" ratio="11" rot="R180"/>
 </element>
+<element name="FID1" library="SparkFun-Retired" package="FIDUCIAL-1.5X3" value="FIDUCIAL1.5X3" x="12" y="50"/>
+<element name="FID2" library="SparkFun-Retired" package="FIDUCIAL-1.5X3" value="FIDUCIAL1.5X3" x="95" y="6"/>
+<element name="FID3" library="SparkFun-Retired" package="FIDUCIAL-1.5X3" value="FIDUCIAL1.5X3" x="59" y="53"/>
+<element name="FID4" library="SparkFun-Retired" package="FIDUCIAL-1.5X3" value="FIDUCIAL1.5X3" x="20" y="75"/>
 </elements>
 <signals>
